File: hardware/steady-hands/PMIC.sch (KiCad schematic (older format))
At the start: 16 parts

Commit message: Feature/bsp structure (#6)
* Adds new BSP src files for new structure since some bsp modules are used multiple times in the drivers

* Adds new BSP src files for new structure since some bsp modules are used multiple times in the drivers

* Adds new BSP src files for new structure since some bsp modules are used multiple times in the drivers

* Adds documentation to bsp src files

* Adds missing bracket
Parts:
- removed J?: USB_B_Micro, symbol Connector:USB_B_Micro
- U?: symbol steady-hands:TPS65721 -> Sij_Power:TPS65721
Changed lines of the file:
@@
 $EndDescr
 $Comp
-L steady-hands:TPS65721 U?
+L Sij_Power:TPS65721 U?
 U 1 1 5F025F79
 P 5150 5650
@@
 	1    0    0    -1
 $EndComp
-$Comp
-L Connector:USB_B_Micro J?
-U 1 1 5EFEB722
-P 2150 2900
-F 0 "J?" H 2207 3367 50  0000 C CNN
-F 1 "USB_B_Micro" H 2207 3276 50  0000 C CNN
-F 2 "" H 2300 2850 50  0001 C CNN
-F 3 "~" H 2300 2850 50  0001 C CNN
-	1    2150 2900
-	1    0    0    -1
-$EndComp

Commit message: Adds symbol library
Parts:
- added J?: USB_B_Micro, symbol Connector:USB_B_Micro
- U?: symbol Sij_Power:TPS65721 -> steady-hands:TPS65721
Changed lines of the file:
@@
 $EndDescr
 $Comp
-L Sij_Power:TPS65721 U?
+L steady-hands:TPS65721 U?
 U 1 1 5F025F79
 P 5150 5650
@@
 	1    0    0    -1
 $EndComp
+$Comp
+L Connector:USB_B_Micro J?
+U 1 1 5EFEB722
+P 2150 2900
+F 0 "J?" H 2207 3367 50  0000 C CNN
+F 1 "USB_B_Micro" H 2207 3276 50  0000 C CNN
+F 2 "" H 2300 2850 50  0001 C CNN
+F 3 "~" H 2300 2850 50  0001 C CNN
+	1    2150 2900
+	1    0    0    -1
+$EndComp
