File: hardware/steady-hands/PMIC.sch (KiCad schematic (older format))
At the start: 16 parts

Commit message: Edits power management
Parts:
- added J?: Conn_01x02, symbol Connector_Generic:Conn_01x02
Connections:
- wire segments 33 -> 40
Other:
- moved on the sheet: J?
Changed lines of the file:
@@
 L Connector:USB_B_Micro J?
 U 1 1 5EFEB722
-P 2150 2900
-F 0 "J?" H 2207 3367 50  0000 C CNN
-F 1 "USB_B_Micro" H 2207 3276 50  0000 C CNN
-F 2 "" H 2300 2850 50  0001 C CNN
-F 3 "~" H 2300 2850 50  0001 C CNN
-	1    2150 2900
+P 2750 2900
+F 0 "J?" H 2807 3367 50  0000 C CNN
+F 1 "USB_B_Micro" H 2807 3276 50  0000 C CNN
+F 2 "" H 2900 2850 50  0001 C CNN
+F 3 "~" H 2900 2850 50  0001 C CNN
+	1    2750 2900
 	1    0    0    -1
 $EndComp
+Wire Wire Line
+	3800 2700 3050 2700
+$Comp
+L power:GND #PWR?
+U 1 1 5EFF0A50
+P 2750 3400
+F 0 "#PWR?" H 2750 3150 50  0001 C CNN
+F 1 "GND" H 2755 3227 50  0000 C CNN
+F 2 "" H 2750 3400 50  0001 C CNN
+F 3 "" H 2750 3400 50  0001 C CNN
+	1    2750 3400
+	1    0    0    -1
+$EndComp
+Wire Wire Line
+	2750 3300 2750 3400
+$Comp
+L Connector_Generic:Conn_01x02 J?
+U 1 1 5EFF19F0
+P 7150 2400
+F 0 "J?" H 7230 2392 50  0000 L CNN
+F 1 "Conn_01x02" H 7230 2301 50  0000 L CNN
+F 2 "" H 7150 2400 50  0001 C CNN
+F 3 "~" H 7150 2400 50  0001 C CNN
+	1    7150 2400
+	1    0    0    -1
+$EndComp
+Wire Wire Line
+	5900 2500 5900 2400
+Wire Wire Line
+	5900 2400 6950 2400
+Connection ~ 5900 2400
+Wire Wire Line
+	6600 2650 6950 2650
+Wire Wire Line
+	6950 2650 6950 2500
+Wire Wire Line
+	6950 2650 6950 2800
+Connection ~ 6950 2650
+$Comp
+L power:GND #PWR?
+U 1 1 5EFF52EA
+P 6950 2800
+F 0 "#PWR?" H 6950 2550 50  0001 C CNN
+F 1 "GND" H 6955 2627 50  0000 C CNN
+F 2 "" H 6950 2800 50  0001 C CNN
+F 3 "" H 6950 2800 50  0001 C CNN
+	1    6950 2800
+	1    0    0    -1
+$EndComp
