File: hardware/steady-hands/PMIC.sch (KiCad schematic (older format))
At the start: 17 parts

Commit message: Adds power management components
Parts:
- removed C?: 22p, symbol Device:C
- removed C? (x2): 4.7u, symbol Device:C
- removed C?: 2.2u, symbol Device:C
- removed C?: 1u, symbol Device:C
- removed L?: 2.2u, symbol Device:L
- removed R?: 680, symbol Device:R
- removed R?: 150, symbol Device:R
- removed R? (x4): R, symbol Device:R
- removed TH?: Thermistor_NTC, symbol Device:Thermistor_NTC
- removed TP?: TestPoint, symbol Connector:TestPoint
- removed U?: TPS65721, Package_DFN_QFN:QFN-32-1EP_4x4mm_P0.4mm_EP2.9x2.9mm, symbol steady-hands:TPS65721
- added C? (x2): 4.7u, symbol Device:C
- added C?: 1u, symbol Device:C
- added D? (x2): LED, symbol Device:LED
- added R? (x2): 1.5k, symbol Device:R
- added R? (x3): R, symbol Device:R
- added SW?: SW_SPDT, symbol Switch:SW_SPDT
- added TH?: 10k, symbol Device:Thermistor
- added U?: BQ24075, symbol Battery_Management:BQ24075
Connections:
- net labels added: CE, CHG, EN1, EN2, OUT, PGOOD, POWER
- wire segments 40 -> 49
Other:
- moved on the sheet: J?
