File: hardware/steady-hands/CapTouch.sch (KiCad schematic (older format))
At the start: 5 parts

Commit message: Adds symbol library
Parts:
- C?: symbol Sij_Touch:CapSense_01x08 -> steady-hands:CapSense_01x08
- U?: symbol Sij_Touch:CPT112S-A02-GM -> steady-hands:CPT112S-A02-GM
Changed lines of the file:
@@
 $EndComp
 $Comp
-L Sij_Touch:CapSense_01x08 C?
+L steady-hands:CapSense_01x08 C?
 U 1 1 5EFBC936
 P 7550 4450
@@
 Connection ~ 3350 4200
 $Comp
-L Sij_Touch:CPT112S-A02-GM U?
+L steady-hands:CPT112S-A02-GM U?
 U 1 1 5EF85C6E
 P 6050 5500

Commit message: Feature/bsp structure (#6)
* Adds new BSP src files for new structure since some bsp modules are used multiple times in the drivers

* Adds new BSP src files for new structure since some bsp modules are used multiple times in the drivers

* Adds new BSP src files for new structure since some bsp modules are used multiple times in the drivers

* Adds documentation to bsp src files

* Adds missing bracket
Parts:
- C?: symbol steady-hands:CapSense_01x08 -> Sij_Touch:CapSense_01x08
Changed lines of the file:
@@
 $EndComp
 $Comp
-L steady-hands:CapSense_01x08 C?
+L Sij_Touch:CapSense_01x08 C?
 U 1 1 5EFBC936
 P 7550 4450
